File: hardware/control_rev3/control_rev3.kicad_sch (KiCad schematic)
At the start: 30 parts, among them J4 Conn_01x07_Pin, J5 Conn_ST_STDC14, P1 Conn_01x03_Pin, P2 Conn_01x03_Pin, P3 Conn_01x03_Pin, P4 Conn_01x03_Pin, SW1 SW_Push, U1 STM32F103C8Tx, Y1 8Mhz

Commit message: Updated to KiCad 9
Parts:
- renumbered C16 to C1, C17 to C2, C18 to C3, C19 to C4, R20 to R2, SW1 to SW2
Changed lines of the file:
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@@
 (kicad_sch
-	(version 20231120)
+	(version 20250114)
 	(generator "eeschema")
-	(generator_version "8.0")
+	(generator_version "9.0")
 	(paper "A4")
 	(title_block
@@
 		(comment 2 "Designed by Abdullah Alsafar")
 	)
+	(text "FS1\n"
+		(exclude_from_sim no)
+		(at 236.22 19.05 0)
+		(effects
+			(font
+				(size 1.27 1.27)
+			)
+			(justify left bottom)
+		)
+	)
+	(text "Servos"
+		(exclude_from_sim no)
+		(at 242.57 73.66 0)
+		(effects
+			(font
+				(size 1.27 1.27)
+			)
+			(justify left bottom)
+		)
+	)
+	(text "Alert system"
+		(exclude_from_sim no)
+		(at 97.155 22.225 0)
+		(effects
+			(font
+				(size 1.27 1.27)
+			)
+			(justify left bottom)
+		)
+	)
+	(text "FS2"
+		(exclude_from_sim no)
+		(at 236.22 42.545 0)
+		(effects
+			(font
+				(size 1.27 1.27)
+			)
+			(justify left bottom)
+		)
+	)
+	(text "TOMAIN"
+		(exclude_from_sim no)
+		(at 196.85 26.035 0)
+		(effects
+			(font
+				(size 1.27 1.27)
+			)
+			(justify left bottom)
+		)
+	)
+	(text "Potentiometers"
+		(exclude_from_sim no)
+		(at 213.36 73.66 0)
+		(effects
+			(font
+				(size 1.27 1.27)
+			)
+			(justify left bottom)
+		)
+	)
+	(text "LED"
+		(exclude_from_sim no)
+		(at 88.392 73.66 0)
+		(effects
+			(font
+				(size 1.27 1.27)
+			)
+			(justify left bottom)
+		)
+	)
 	(junction
 		(at 165.1 64.77)
@@
 		)
 	)
-	(text "FS1\n"
-		(exclude_from_sim no)
-		(at 236.22 19.05 0)
-		(effects
-			(font
-				(size 1.27 1.27)
-			)
-			(justify left bottom)
-		)
-	)
-	(text "Servos"
-		(exclude_from_sim no)
-		(at 242.57 73.66 0)
-		(effects
-			(font
-				(size 1.27 1.27)
-			)
-			(justify left bottom)
-		)
-	)
-	(text "Alert system"
-		(exclude_from_sim no)
-		(at 97.155 22.225 0)
-		(effects
-			(font
-				(size 1.27 1.27)
-			)
-			(justify left bottom)
-		)
-	)
-	(text "FS2"
-		(exclude_from_sim no)
-		(at 236.22 42.545 0)
-		(effects
-			(font
-				(size 1.27 1.27)
-			)
-			(justify left bottom)
-		)
-	)
-	(text "TOMAIN"
-		(exclude_from_sim no)
-		(at 196.85 26.035 0)
-		(effects
-			(font
-				(size 1.27 1.27)
-			)
-			(justify left bottom)
-		)
-	)
-	(text "Potentiometers"
-		(exclude_from_sim no)
-		(at 213.36 73.66 0)
-		(effects
-			(font
-				(size 1.27 1.27)
-			)
-			(justify left bottom)
-		)
-	)
-	(text "LED"
-		(exclude_from_sim no)
-		(at 88.392 73.66 0)
-		(effects
-			(font
-				(size 1.27 1.27)
-			)
-			(justify left bottom)
-		)
-	)
 	(label "SWCLK"
 		(at 129.54 158.75 180)
-		(fields_autoplaced yes)
 		(effects
 			(font
@@
 	(label "SWDIO"
 		(at 186.69 102.87 180)
-		(fields_autoplaced yes)
 		(effects
 			(font
@@
 	(label "~{RST}"
 		(at 129.54 153.67 180)
-		(fields_autoplaced yes)
 		(effects
 			(font
@@
 	(label "~{RST}"
 		(at 138.43 62.23 0)
-		(fields_autoplaced yes)
 		(effects
 			(font
@@
 	(label "SWDIO"
 		(at 129.54 161.29 180)
-		(fields_autoplaced yes)
 		(effects
 			(font
@@
 	(label "SWCLK"
 		(at 186.69 105.41 180)
-		(fields_autoplaced yes)
 		(effects
 			(font
@@
 		(dnp no)
 		(fields_autoplaced yes)
-		(property "Reference" "#PWR023"
+		(property "Reference" "#PWR042"
 			(at 123.19 99.06 0)
 			(effects
@@
 		(dnp no)
 		(fields_autoplaced yes)
-		(property "Reference" "#PWR024"
+		(property "Reference" "#PWR021"
 			(at 114.3 68.58 0)
 			(effects
@@
 		(dnp no)
 		(fields_autoplaced yes)
-		(property "Reference" "R20"
+		(property "Reference" "R2"
 			(at 134.62 57.1499 0)
 			(effects
@@
 		(on_board yes)
 		(dnp no)
-		(property "Reference" "#PWR028"
+		(property "Reference" "#PWR023"
 			(at 157.48 66.04 0)
 			(effects
@@
 		(dnp no)
 		(fields_autoplaced yes)
-		(property "Reference" "#PWR023"
+		(property "Reference" "#PWR020"
 			(at 114.3 82.55 0)
 			(effects
@@
 		(on_board yes)
 		(dnp no)
-		(property "Reference" "C16"
+		(property "Reference" "C1"
 			(at 157.48 30.48 90)
 			(effects
@@
 		(on_board yes)
 		(dnp no)
-		(property "Reference" "C18"
+		(property "Reference" "C3"
 			(at 154.94 48.26 90)
 			(effects
@@
 		(dnp no)
 		(fields_autoplaced yes)
-		(property "Reference" "#PWR023"
+		(property "Reference" "#PWR026"
 			(at 127 109.22 0)
 			(effects
@@
 		(on_board yes)
 		(dnp no)
-		(property "Reference" "C17"
+		(property "Reference" "C2"
 			(at 154.94 41.91 90)
 			(effects
@@
 		(dnp no)
 		(fields_autoplaced yes)
-		(property "Reference" "SW1"
+		(property "Reference" "SW2"
 			(at 119.38 54.61 0)
 			(effects
@@
 		(on_board yes)
 		(dnp no)
-		(property "Reference" "C19"
+		(property "Reference" "C4"
 			(at 167.64 54.61 90)
 			(effects
@@
 		(at 45.72 147.32)
 		(size 24.13 17.78)
+		(exclude_from_sim no)
+		(in_bom yes)
+		(on_board yes)
+		(dnp no)
 		(fields_autoplaced yes)
 		(stroke
@@
 		)
 		(instances
-			(project "control"
+			(project "control_rev3"
 				(path "/e7781990-9217-47e0-bccf-d5b77eec6675"
 					(page "2")
@@
 		)
 	)
+	(embedded_fonts no)
 )
