File: hardware/control_rev3/v_regs.kicad_sch (KiCad schematic)
At the start: 25 parts, among them J1 Conn_01x02_Pin, J3 Conn_01x02_Pin

Commit message: Updated to KiCad 9
Parts:
- R4: value 33.2k -> 33.2k
